Commit message: trajecotory for heart is working!

File: urdf/arms.urdf (robot description, URDF)
Before this commit: robot penarm, 4 links, 3 joints
Links:
- added link gripper_arm; visual cylinder length=0.1 radius=0.05
Joints:
- removed joint lower_arm_end_effector
- added joint gripper_arm_end_effector: type fixed, parent gripper_arm, child end_effector, origin xyz=0.1 0 0.0 rpy=0 0 0
- added joint lower_arm_gripper_arm: type revolute, parent lower_arm, child gripper_arm, origin xyz=1.0 0 0.0 rpy=0 0 0, axis 0 0 1, limit lower=-3.142 upper=3.142 effort=100 velocity=100
